File: hardware_design/electrical/OdinsEye/OdinsEye.kicad_sch (KiCad schematic)
At the start: 17 parts

Commit message: Add connector design
Parts:
- J1: renamed from J?; value BATT_Male -> BATT_JST-CH2.5-2P_Male
- J10: renamed from J?; value AS5600_devboard_1_Female -> AS5600_devboard_1_JST-XH2.5-3P_Female
- J11: renamed from J?; value AS5600_devboard_2_Male -> AS5600_devboard_2_JST-XH2.5-4P_Male
- J12: renamed from J?; value AS5600_devboard_2_Female -> AS5600_devboard_2_JST-XH2.5-4P_Female
- J2: renamed from J?; value BATT_Female -> BATT_JST-CH2.5-2P_Female
- J3: renamed from J?; value GT-U7_devboard_Male -> GT-U7_devboard_JST-XH2.5-SIDE-5P_Male
- J4: renamed from J?; value GT-U7_devboard_Female -> GT-U7_devboard_JST-XH2.5-5P_Female
- J5: renamed from J?; value GC9A01A_01.28LCD_Male -> GC9A01A_01.28LCD_JST-PH2.0-SIDE-8P_Male
- J6: renamed from J?; value GC9A01A_01.28LCD_Female -> GC9A01A_01.28LCD_JST-PH2.0-8P_Female
- J7: renamed from J?; value WS2812_24O_Male -> WS2812_24O_JST-XH2.5-SIDE-3P_Male
- J8: renamed from J?; value WS2812_24O_Female -> WS2812_24O_JST-XH2.5-3P_Female
- J9: renamed from J?; value AS5600_devboard_1_Male -> AS5600_devboard_1_JST-XH2.5-3P_Male
- gave numbers to parts that had none: 5
Connections:
- net GND: now also U1.14 (GND); no longer J1.2 (Pin_2), U1.2 (GND)
- new net: J1.2 (Pin_2), U1.2 (GND)
Other:
- moved on the sheet: J10, J2, J3, U2
